Commit message: added camera plugins

File: bot_description/urdf/bot.urdf (robot description, URDF)
Before this commit: robot my_bot, 12 links, 11 joints
Links:
- added link camera_depth
- added link camera_depth_link; visual box size=0.010 0.03 0.03; visual cylinder length=0.1 radius=0.002
- added link camera_link; visual box size=0.010 0.03 0.03; visual cylinder length=0.1 radius=0.002
- added link camera_link_optical
Joints:
- added joint camera_1_joint: type fixed, parent chassis, child camera_link, origin xyz=0 -0.25 0.08 rpy=0 0 -1.57
- added joint camera_2_joint: type fixed, parent chassis, child camera_depth_link, origin xyz=0 -0.25 0.08 rpy=0 0 -1.57
- added joint camera_depth_joint: type fixed, parent camera_depth_link, child camera_depth, origin xyz=0 0 0 rpy=${-pi/2} 0 ${-pi/2}
- added joint camera_optical_joint: type fixed, parent camera_link, child camera_link_optical, origin xyz=0 0 0 rpy=${-pi/2} 0 ${-pi/2}

Commit message: modified

File: bot_description/urdf/bot.urdf (robot description, URDF)
Before this commit: robot my_bot, 16 links, 15 joints
Links:
- removed link camera_link
- removed link camera_link_optical
Joints:
- removed joint camera_1_joint
- removed joint camera_optical_joint
